File: pcb/Tiny_Thinker.kicad_pcb (KiCad board)
At the start: 4 copper layers, 118.9 x 69.3 mm, 47 parts, among them J1 Conn_02x20_Odd_Even, J2 Conn_02x20_Odd_Even, J3 SWD, J4 SPI1, J5 I2C1_A, J6 I2C1_B, J7 Conn_02x20_Odd_Even, J8 USB_C_Receptacle_USB2.0_16P, SW1 SW_Push, SW2 SW_SPDT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

Commit message: checkpoint
Parts:
- removed J7: Conn_02x20_Odd_Even, Connector_PinHeader_2.54mm:PinHeader_2x20_P2.54mm_Vertical
- C10, C11: value 10pF -> 1uF
- C14: value 4.7uF -> 10pF
- C15: value 100nF -> 10pF
- C5: value 10uF -> 100nF; footprint Capacitor_SMD:C_0603_1608Metric -> Capacitor_SMD:C_0402_1005Metric
- C6: value 10nF -> 10uF; footprint Capacitor_SMD:C_0402_1005Metric -> Capacitor_SMD:C_0603_1608Metric
- C7: value 1uF -> 100nF
- C8: value 1uF -> 4.7uF
- C9: value 100nF -> 10nF
- moved J2 125.2 mm to (202.2, 76.9), turned to 0 degrees
- moved J4 84.4 mm to (186.5, 56.0), turned to 0 degrees
- moved J3 64.4 mm to (180.6, 79.8), turned to 0 degrees
- moved C4 45.6 mm to (144.2, 97.8), turned to -90 degrees
- moved C2 45.0 mm to (133.8, 109.0), turned to 180 degrees
- moved C8 43.7 mm to (139.2, 109.0), turned to -90 degrees
- moved C10 42.9 mm to (128.2, 107.5), turned to 180 degrees
- moved C11 42.6 mm to (128.3, 109.0), turned to 180 degrees
- moved C9 41.4 mm to (129.2, 103.2), turned to 90 degrees
- moved R2 38.7 mm to (158.2, 111.5)
- moved C13 38.7 mm to (155.5, 116.0)
- moved U2 38.5 mm to (150.2, 116.2)
- moved C12 38.4 mm to (150.0, 110.5)
- moved D1 38.2 mm to (158.2, 114.2)
- moved Y1 36.6 mm to (124.4, 99.5)
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Connections:
- C10 pad 1: /HSE_IN -> +3.3VA
- C11 pad 1: /HSE_OUT -> +3.3V
- C14 pad 1: /VCAP_1 -> /HSE_IN
- C15 pad 1: +3.3V -> /HSE_OUT
- C6 pad 1: +3.3VA -> +3.3V
- C7 pad 1: +3.3VA -> /NRST
- C8 pad 1: +3.3V -> /VCAP_1
- C9 pad 1: /NRST -> +3.3VA
- D2 pad 1: Net-(D2-I/O1-Pad1) -> /USB_D-
- D2 pad 3: Net-(D2-I/O2-Pad3) -> /USB_D+
- J8 pad A6: Net-(D2-I/O2-Pad3) -> /USB_D+
- J8 pad A7: Net-(D2-I/O1-Pad1) -> /USB_D-
- J8 pad B6: Net-(D2-I/O2-Pad3) -> /USB_D+
- J8 pad B7: Net-(D2-I/O1-Pad1) -> /USB_D-
Routing:
- net GND: track 34.9 -> 11.2 mm, vias 25 -> 0
- net /BOOT0: track 25.5 -> 3.23 mm
- net +VBUS: track 0.00 -> 18.2 mm
- net /SWDIO: track 13.5 -> 0.00 mm
- net /SWCLK: track 11.0 -> 0.00 mm
- net /NRST: track 14.3 -> 4.28 mm
- net /USBCC1: track 0.00 -> 8.46 mm
- net /USBCC2: track 0.00 -> 8.04 mm
- net +3.3V: track 20.0 -> 13.1 mm
- net /HSE_IN: track 4.14 -> 8.49 mm
- net +3.3VA: track 7.80 -> 3.51 mm
- net /HSE_OUT: track 1.91 -> 6.08 mm
- net /SW_BOOT0: track 4.07 -> 0.00 mm
- net +VBUSF: track 0.00 -> 3.05 mm
- net /PWR_LED_K: track 2.20 -> 0.00 mm
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- removed copper zone on F.Cu, net +3.3V
- removed copper zone on F.Cu, net +VBUSF
- removed copper zone on F.Cu, net GND
- removed copper zone on In1.Cu, net GND
- removed copper zone on In2.Cu, net GND
Other:
- board outline removed
- board text removed: "->"
- board text removed: "BOOT"

Commit message: checkpoint
Parts:
- added J7: CAN1, Connector_PinHeader_2.54mm:PinHeader_1x04_P2.54mm_Vertical, F.Cu at (131.5, 82.5)
- moved J4 76.8 mm to (141.3, 118.0), turned to -90 degrees
- moved J6 47.3 mm to (143.0, 86.5), turned to 90 degrees
- moved J5 42.3 mm to (143.0, 82.5), turned to 90 degrees
- moved J3 24.0 mm to (156.7, 82.7)
- moved SW2 13.1 mm to (123.8, 82.1), turned to 180 degrees
- moved R1 7.74 mm to (123.0, 85.8), turned to -90 degrees
- moved SW1 1.81 mm to (124.0, 90.6)
- moved C7 1.72 mm to (125.8, 93.1)
- moved C14 0.97 mm to (127.3, 97.5)
- moved Y1 0.97 mm to (124.7, 98.6)
- moved C15 0.96 mm to (127.2, 99.7)
Connections:
- D2 pad 1: /USB_D- -> Net-(D2-I/O1-Pad1)
- D2 pad 3: /USB_D+ -> Net-(D2-I/O2-Pad3)
- J8 pad A6: /USB_D+ -> Net-(D2-I/O2-Pad3)
- J8 pad A7: /USB_D- -> Net-(D2-I/O1-Pad1)
- J8 pad B6: /USB_D+ -> Net-(D2-I/O2-Pad3)
- J8 pad B7: /USB_D- -> Net-(D2-I/O1-Pad1)
Routing:
- net GND: track 11.2 -> 39.4 mm, vias 0 -> 25
- net /SWDIO: track 0.00 -> 22.2 mm
- net /SWCLK: track 0.00 -> 20.9 mm
- net /I2C1_SCL: track 0.00 -> 20.4 mm
- net /I2C1_SDA: track 0.00 -> 18.5 mm
- net /BOOT0: track 3.23 -> 20.1 mm
- net /CAN1_RX: track 0.00 -> 13.9 mm
- net /CAN1_TX: track 0.00 -> 13.9 mm
- net /NRST: track 4.28 -> 15.9 mm
- net Net-(D2-I/O2-Pad3): track 0.00 -> 5.70 mm
- net /USB_D+: track 10.4 -> 4.75 mm
- net Net-(D2-I/O1-Pad1): track 0.00 -> 5.02 mm
- net /USB_D-: track 9.76 -> 4.75 mm
- net /SW_BOOT0: track 0.00 -> 1.81 mm
- net (no net): vias 2 -> 0
- added copper zone on In1.Cu, net GND
- added copper zone on In2.Cu, net GND
Other:
- board outline added: 60 x 41.8 mm

Commit message: checkpoint
Parts:
- moved J4 9.00 mm to (132.3, 118.2)
Connections:
- D2 pad 1: Net-(D2-I/O1-Pad1) -> /USB_D-
- J8 pad A6: Net-(D2-I/O2-Pad3) -> /USB_D+
- J8 pad A7: Net-(D2-I/O1-Pad1) -> /USB_D-
- J8 pad B6: Net-(D2-I/O2-Pad3) -> /USB_D+
- J8 pad B7: Net-(D2-I/O1-Pad1) -> /USB_D-
Routing:
- net Net-(D2-I/O2-Pad3): track 5.70 -> 0.00 mm
- net /USB_D+: track 4.75 -> 10.4 mm
- net +3.3V: track 13.1 -> 18.6 mm, vias 0 -> 4
- net Net-(D2-I/O1-Pad1): track 5.02 -> 0.00 mm
- net /USB_D-: track 4.75 -> 9.73 mm
- net GND: track 39.4 -> 40.5 mm, vias 25 -> 26
- net +VBUS: track 18.2 -> 17.6 mm
- added copper zone on B.Cu, net +3.3V
