File: pcb/_autosave-Tiny_Thinker.kicad_sch (KiCad schematic)
At the start: 51 parts, among them J1 Conn_02x20_Odd_Even, J10 ADC1_A, J11 TIM3_A, J12 TIM3_B, J2 Conn_02x20_Odd_Even, J3 SWD, J4 SPI1, J5 I2C1_A, J6 I2C1_B, J7 CAN1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

Commit message: rough layout done
Parts:
- removed J2: Conn_02x20_Odd_Even, Connector_PinHeader_2.54mm:PinHeader_2x20_P2.54mm_Vertical, symbol Connector_Generic:Conn_02x20_Odd_Even
- added J13: TIM3_A, Connector_PinHeader_2.54mm:PinHeader_1x04_P2.54mm_Vertical, symbol Connector:Conn_01x04_Pin
- added J14: TIM3_B, Connector_PinHeader_2.54mm:PinHeader_1x04_P2.54mm_Vertical, symbol Connector:Conn_01x04_Pin
Connections:
- net ADC1_IN19 is gone; now on net ADC1_IN9: J10.1 (Pin_1)
- net GND: now also J13.2 (Pin_2), J13.4 (Pin_4), J14.1 (Pin_1), J14.3 (Pin_3)
- net TIM2_CH1: now also J13.1 (Pin_1)
- net TIM2_CH2: now also J14.2 (Pin_2)
- net TIM2_CH3: now also J13.3 (Pin_3)
- net TIM2_CH4: now also J14.4 (Pin_4)
- net TIM3_CH1: now also J11.1 (Pin_1); no longer J11.3 (Pin_3)
- net TIM3_CH2: now also J12.2 (Pin_2); no longer J12.4 (Pin_4)
- net TIM3_CH3: now also J11.3 (Pin_3); no longer J11.1 (Pin_1)
- net TIM3_CH4: now also J12.4 (Pin_4); no longer J12.2 (Pin_2)
Other:
- moved on the sheet: J1
