File: pcb/_autosave-Tiny_Thinker.kicad_sch (KiCad schematic)
At the start: 42 parts, among them J2 PERIPHERALS, J3 ADC_TIM, J8 USB_C_Receptacle_USB2.0_16P, SW1 SW_Push, SW2 SW_SPDT, U1 STM32F446RET6, U2 AMS1117-3.3, Y1 16MHz

Commit message: routed peripherals
Connections:
- net +3.3V: now also J2.10 (Pin_10), J2.18 (Pin_18), J2.9 (Pin_9), J3.37 (Pin_37), J3.40 (Pin_40); no longer J2.13 (Pin_13), J2.14 (Pin_14), J2.25 (Pin_25), J2.29 (Pin_29)
- net CAN1_RX: now also J2.32 (Pin_32); no longer J2.24 (Pin_24)
- net CAN1_TX: now also J2.34 (Pin_34); no longer J2.26 (Pin_26)
- net GND: now also J2.16 (Pin_16), J2.36 (Pin_36), J2.7 (Pin_7), J3.38 (Pin_38), J3.39 (Pin_39); no longer J2.10 (Pin_10), J2.11 (Pin_11), J2.12 (Pin_12), J2.23 (Pin_23), J2.31 (Pin_31), J2.32 (Pin_32)
- net I2C1_SCL: now also J2.23 (Pin_23), J2.24 (Pin_24); no longer J2.15 (Pin_15), J2.16 (Pin_16)
- net I2C1_SDA: now also J2.25 (Pin_25), J2.26 (Pin_26); no longer J2.17 (Pin_17), J2.18 (Pin_18)
- net SPI1_MISO: now also J2.15 (Pin_15); no longer J2.7 (Pin_7)
- net SPI1_MOSI: now also J2.17 (Pin_17); no longer J2.9 (Pin_9)
- net SPI1_NSS: now also J2.11 (Pin_11); no longer J2.3 (Pin_3)
- net SPI1_SCK: now also J2.13 (Pin_13); no longer J2.5 (Pin_5)
- net SWCLK: now also J2.5 (Pin_5); no longer J2.6 (Pin_6)
- net SWDIO: now also J2.3 (Pin_3); no longer J2.4 (Pin_4)
- net USB_D+: now also D2.3 (I/O2), J8.A6 (D+), J8.B6 (D+)
- net USB_D-: now also D2.1 (I/O1), J8.A7 (D-), J8.B7 (D-)
- net SPI2_NSS: now reaches U1.33 (PB12)
- net SPI2_SCK: now reaches U1.34 (PB13)
- net SPI2_MISO: now reaches U1.35 (PB14)
- net SPI2_MOSI: now reaches U1.36 (PB15)
- no-connect marks 25 -> 21
