File: pcb/_autosave-Tiny_Thinker.kicad_pcb (KiCad board)
At the start: 4 copper layers, 65 x 63.1 mm, 42 parts, among them J2 PERIPHERALS, J3 ADC_TIM, J8 USB_C_Receptacle_USB2.0_16P, SW1 SW_Push, SW2 SW_SPDT, U1 STM32F446RET6, U2 AMS1117-3.3, Y1 16MHz

Commit message: routed peripherals
Parts:
- moved C3 0.28 mm to (132.7, 93.8)
- moved C6 0.28 mm to (132.7, 92.2)
Connections:
- J2 pad 10: GND -> +3.3V
- J2 pad 11: GND -> /SPI1_NSS
- J2 pad 12: GND -> unconnected-(J2-Pin_12-Pad12)
- J2 pad 13: +3.3V -> /SPI1_SCK
- J2 pad 14: +3.3V -> unconnected-(J2-Pin_14-Pad14)
- J2 pad 15: /I2C1_SCL -> /SPI1_MISO
- J2 pad 16: /I2C1_SCL -> GND
- J2 pad 17: /I2C1_SDA -> /SPI1_MOSI
- J2 pad 18: /I2C1_SDA -> +3.3V
- J2 pad 23: GND -> /I2C1_SCL
- J2 pad 24: /CAN1_RX -> /I2C1_SCL
- J2 pad 25: +3.3V -> /I2C1_SDA
- J2 pad 26: /CAN1_TX -> /I2C1_SDA
- J2 pad 29: +3.3V -> unconnected-(J2-Pin_29-Pad29)
- J2 pad 3: /SPI1_NSS -> unconnected-(J2-Pin_3-Pad3)
- J2 pad 31: GND -> unconnected-(J2-Pin_31-Pad31)
- J2 pad 32: GND -> /CAN1_RX
- J2 pad 34: unconnected-(J2-Pin_34-Pad34) -> /CAN1_TX
- J2 pad 36: unconnected-(J2-Pin_36-Pad36) -> GND
- J2 pad 5: /SPI1_SCK -> unconnected-(J2-Pin_5-Pad5)
- J2 pad 7: /SPI1_MISO -> GND
- J2 pad 9: /SPI1_MOSI -> +3.3V
- J3 pad 1: /TIM3_CH4 -> +VBUSF
- J3 pad 12: +3.3V -> /TIM3_CH1
- J3 pad 13: /ADC1_IN9 -> +3.3V
- J3 pad 16: /ADC1_IN8 -> +3.3V
- J3 pad 17: /ADC1_IN15 -> /ADC1_IN9
- J3 pad 20: /ADC1_IN14 -> /ADC1_IN8
- J3 pad 21: +3.3V -> /ADC1_IN15
- J3 pad 24: +3.3V -> /ADC1_IN14
- J3 pad 25: /TIM2_CH4 -> +3.3V
- J3 pad 28: /TIM2_CH3 -> +3.3V
- J3 pad 29: /TIM2_CH2 -> /TIM2_CH4
- J3 pad 32: /TIM2_CH1 -> /TIM2_CH3
- J3 pad 33: unconnected-(J3-Pin_33-Pad33) -> /TIM2_CH2
- J3 pad 34: unconnected-(J3-Pin_34-Pad34) -> GND
- J3 pad 35: unconnected-(J3-Pin_35-Pad35) -> GND
- J3 pad 36: unconnected-(J3-Pin_36-Pad36) -> /TIM2_CH1
- J3 pad 37: unconnected-(J3-Pin_37-Pad37) -> +3.3V
- J3 pad 38: unconnected-(J3-Pin_38-Pad38) -> GND
- J3 pad 39: unconnected-(J3-Pin_39-Pad39) -> GND
- J3 pad 4: /TIM3_CH3 -> +VBUSF
- J3 pad 40: unconnected-(J3-Pin_40-Pad40) -> +3.3V
- J3 pad 5: /TIM3_CH2 -> /TIM3_CH4
- J3 pad 8: /TIM3_CH1 -> /TIM3_CH3
- J3 pad 9: +3.3V -> /TIM3_CH2
- U1 pad 33: unconnected-(U1-PB12-Pad33) -> /SPI2_NSS
- U1 pad 34: unconnected-(U1-PB13-Pad34) -> /SPI2_SCK
- U1 pad 35: unconnected-(U1-PB14-Pad35) -> /SPI2_MISO
- U1 pad 36: unconnected-(U1-PB15-Pad36) -> /SPI2_MOSI
Routing:
- net GND: track 79.3 -> 35.6 mm, vias 46 -> 35
- net /CAN1_TX: track 4.89 -> 34.0 mm
- net /SPI1_MOSI: track 0.00 -> 27.6 mm
- net /CAN1_RX: track 5.09 -> 32.1 mm
- net /SPI1_MISO: track 0.00 -> 26.5 mm
- net /SPI1_SCK: track 0.00 -> 25.7 mm
- net /SPI1_NSS: track 0.00 -> 24.8 mm
- net /I2C1_SDA: track 2.43 -> 26.2 mm
- net +VBUSF: track 6.65 -> 28.9 mm
- net /SWDIO: track 5.86 -> 27.2 mm
- net /I2C1_SCL: track 2.18 -> 23.5 mm
- net /SPI2_NSS: track 0.00 -> 8.05 mm, vias 0 -> 1
- net /SPI2_MISO: track 0.00 -> 7.80 mm, vias 0 -> 1
- net /SPI2_SCK: track 0.00 -> 7.58 mm, vias 0 -> 1
- net +3.3V: track 30.2 -> 22.6 mm, vias 18 -> 14
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