File: pcb/_autosave-Tiny_Thinker.kicad_pcb (KiCad board)
At the start: 4 copper layers, 65 x 63.1 mm, 46 parts, among them J2 PERIPHERALS, J3 ADC_TIM, J8 USB_C_Receptacle_USB2.0_16P, SW1 SW_Push, SW2 SW_SPDT, U1 STM32F446RET6, U2 AMS1117-3.3, U3 TPS2116DRL, Y1 16MHz

Commit message: changed dimensions to be whole numbers
Parts:
- moved H1 8.90 mm to (95.5, 65.0)
Routing:
- net GND: vias 75 -> 74
Other:
- board size 65 x 63.1 mm -> 67.9 x 73.7 mm
Changed lines of the file:
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@@
 	(footprint "MountingHole:MountingHole_2.2mm_M2"
 		(layer "F.Cu")
-		(at 97.42502 73.7)
+		(at 95.50002 65.015)
 		(descr "Mounting Hole 2.2mm, M2, no annular, generated by kicad-footprint-generator mountinghole.py")
 		(tags "mountinghole M2")
@@
 			(remove_unused_layers yes)
 			(keep_end_layers yes)
-			(zone_layer_connections "In1.Cu" "In2.Cu")
+			(zone_layer_connections)
 			(net 1 "GND")
 			(pinfunction "SHIELD")
@@
 			(remove_unused_layers yes)
 			(keep_end_layers yes)
-			(zone_layer_connections "In1.Cu" "In2.Cu")
+			(zone_layer_connections)
 			(net 1 "GND")
 			(pinfunction "SHIELD")
@@
 			(remove_unused_layers yes)
 			(keep_end_layers yes)
-			(zone_layer_connections "In1.Cu" "In2.Cu")
+			(zone_layer_connections)
 			(net 1 "GND")
 			(pinfunction "SHIELD")
@@
 			(remove_unused_layers yes)
 			(keep_end_layers yes)
-			(zone_layer_connections "In1.Cu" "In2.Cu")
+			(zone_layer_connections)
 			(net 1 "GND")
 			(pinfunction "SHIELD")
@@
 	)
 	(gr_line
-		(start 94.425 130.765)
-		(end 94.425 73.685)
+		(start 94.425 134.725)
+		(end 94.425 69.725)
 		(stroke
 			(width 0.05)
-			(type default)
+			(type solid)
 		)
 		(layer "Edge.Cuts")
 	)
 	(gr_line
-		(start 97.425 133.765)
-		(end 156.425 133.765)
+		(start 94.425 134.725)
+		(end 159.425 134.725)
 		(stroke
 			(width 0.05)
@@
 		(layer "Edge.Cuts")
 	)
-	(gr_arc
-		(start 94.425 73.685)
-		(mid 95.30368 71.56368)
-		(end 97.425 70.685)
+	(gr_line
+		(start 94.425 69.725)
+		(end 159.425 69.725)
 		(stroke
 			(width 0.05)
@@
 		(layer "Edge.Cuts")
 	)
-	(gr_line
-		(start 97.425 70.685)
-		(end 156.425 70.685)
+	(gr_arc
+		(start 91.5 65)
+		(mid 92.671573 62.171573)
+		(end 95.5 61)
 		(stroke
 			(width 0.05)
@@
 	)
 	(gr_line
-		(start 159.425 73.685)
-		(end 159.425 130.765)
+		(start 159.425 69.725)
+		(end 159.425 134.725)
 		(stroke
 			(width 0.05)
-			(type default)
+			(type solid)
 		)
 		(layer "Edge.Cuts")
@@
 	)
 	(via
-		(at 158 108)
-		(size 0.9)
-		(drill 0.4)
-		(layers "F.Cu" "B.Cu")
-		(remove_unused_layers yes)
-		(keep_end_layers yes)
-		(free yes)
-		(zone_layer_connections "In1.Cu" "In2.Cu")
-		(net 1)
-	)
-	(via
 		(at 152.775 107.855)
 		(size 0.7)
@@
 	)
 	(segment
-		(start 114.8 123.7)
-		(end 114.8 128.44)
+		(start 133.8 104.4)
+		(end 133.8 104.7)
 		(width 0.3)
 		(layer "F.Cu")
@@
 	)
 	(segment
-		(start 114.8 128.44)
-		(end 113.475 129.765)
+		(start 133.4 104)
+		(end 133.8 104.4)
 		(width 0.3)
 		(layer "F.Cu")
@@
 	)
 	(segment
-		(start 133.8 104.7)
-		(end 114.8 123.7)
+		(start 114.75 123.75)
+		(end 114.75 128.49)
 		(width 0.3)
 		(layer "F.Cu")
@@
 	)
 	(segment
-		(start 133.8 104.4)
-		(end 133.8 104.7)
+		(start 114.75 128.49)
+		(end 113.475 129.765)
 		(width 0.3)
 		(layer "F.Cu")
@@
 	)
 	(segment
-		(start 133.4 104)
-		(end 133.8 104.4)
+		(start 133.8 104.7)
+		(end 114.75 123.75)
 		(width 0.3)
 		(layer "F.Cu")
